File: board/hw-USB-RF.kicad_pcb (KiCad board)
At the start: 2 copper layers, 45 x 16 mm, 20 parts, among them J1 USB_OTG, U1 CMT2210L, U2 SPX3819, U3 ATSAMD11C14A-SS, X1 SWD, X2 SG-210STF

Commit message: WIP
Parts:
- removed L2: 15nH, Inductor_SMD:L_0805_2012Metric
- removed X2: SG-210STF, Oscillator:Oscillator_SMD_SeikoEpson_SG210-4Pin_2.5x2.0mm
- added C9: 1u, Capacitor_SMD:C_0805_2012Metric, F.Cu at (123.0, 97.0)
- added Y1: 12MHz, Crystal:Crystal_SMD_3225-4Pin_3.2x2.5mm, F.Cu at (121.0, 89.0)
- C4, C5: value 100n -> 15p
- C6: value 10n -> 100n
- C7: value 1u -> 100n
- C8: value 100n -> 10n
- moved C4 19.6 mm to (118.0, 89.0)
- moved C2 18.1 mm to (138.0, 91.0)
- moved C6 14.7 mm to (135.0, 91.0), turned to 270 degrees
- moved C8 14.7 mm to (123.0, 99.5), turned to 0 degrees
- moved TP1 13.2 mm to (144.5, 88.5), turned to 270 degrees
- moved D1 9.80 mm to (136.8, 94.0), turned to 0 degrees
- moved R1 9.29 mm to (136.8, 96.5)
- moved C5 5.59 mm to (124.0, 89.0), turned to 90 degrees
- moved AE1 3.50 mm to (150.0, 94.0)
- moved C7 2.50 mm to (123.0, 94.5)
- moved C3 2.06 mm to (141.5, 98.5)
- moved C1 1.50 mm to (149.5, 90.5)
- moved L1 1.17 mm to (148.0, 88.0), turned to 0 degrees
Connections:
- C2 pad 1: +3V3 -> GND
- C2 pad 2: GND -> +3V3
- C3 pad 2: /26MHZ -> /23M138
- C4 pad 2: +3V3 -> Net-(C4-Pad2)
- C5 pad 1: Net-(C5-Pad1) -> GND
- C5 pad 2: GND -> Net-(C5-Pad2)
- C6 pad 1: Net-(C6-Pad1) -> +3V3
- C7 pad 1: +3V3 -> Net-(C7-Pad1)
- C8 pad 1: +3V3 -> Net-(C8-Pad1)
- D1 pad 1: GND -> Net-(D1-Pad1)
- D1 pad 2: Net-(D1-Pad2) -> /LED
- J1 pad 4: (no net) -> Net-(J1-Pad4)
- R1 pad 1: /LED -> Net-(D1-Pad1)
- R1 pad 2: Net-(D1-Pad2) -> GND
- U1 pad 4: (no net) -> GND
- U1 pad 6: Net-(L2-Pad2) -> (no net)
- U1 pad 7: Net-(L2-Pad1) -> (no net)
- U2 pad 4: Net-(C6-Pad1) -> Net-(C8-Pad1)
- U3 pad 14: (no net) -> Net-(U3-Pad14)
- U3 pad 2: /26MHZ -> Net-(C5-Pad2)
- U3 pad 3: /OSC_EN -> Net-(C4-Pad2)
- U3 pad 4: (no net) -> /23M138
- U3 pad 5: (no net) -> Net-(U3-Pad5)
- U3 pad 6: Net-(C5-Pad1) -> Net-(C7-Pad1)
Routing:
- net /26MHZ: track 31.1 -> 0.00 mm, vias 2 -> 0
- net /23M138: track 0.00 -> 18.8 mm
- net Net-(C4-Pad2): track 0.00 -> 9.51 mm
- net /LED: track 13.3 -> 20.4 mm, vias 0 -> 2
- net GND: track 11.3 -> 17.4 mm, vias 14 -> 15
- net Net-(C5-Pad2): track 0.00 -> 5.60 mm
- net Net-(L2-Pad2): track 3.84 -> 0.00 mm
- net Net-(L2-Pad1): track 3.59 -> 0.00 mm
- net /OSC_EN: track 3.57 -> 0.00 mm
- net Net-(C5-Pad1): track 2.88 -> 0.00 mm
- net Net-(C7-Pad1): track 0.00 -> 2.88 mm
- net Net-(D1-Pad1): track 0.00 -> 2.50 mm
- net Net-(C8-Pad1): track 0.00 -> 2.48 mm
- net Net-(C6-Pad1): track 2.48 -> 0.00 mm
- net Net-(D1-Pad2): track 2.12 -> 0.00 mm
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Other:
- board size 45 x 16 mm -> 41 x 16 mm
- board text added: "USB-RF"
- board text added: "v1.3"
- board text removed: "USB-RF v1.2"

Commit message: WIP
Parts:
- turned C4 to 90 degrees
- turned C5 to 270 degrees
Connections:
- net /23M138 renamed /27M138
- Y1 pad 1: GND -> Net-(C5-Pad2)
- Y1 pad 2: Net-(C5-Pad2) -> GND
- Y1 pad 3: GND -> Net-(C4-Pad2)
- Y1 pad 4: Net-(C4-Pad2) -> GND
Routing:
- net Net-(C4-Pad2): track 9.51 -> 0.00 mm
- net GND: track 17.4 -> 10.0 mm, vias 15 -> 13
- net Net-(C5-Pad2): track 5.60 -> 0.00 mm
Other:
- board text added: "v1.4"
- board text removed: "v1.3"
